Commit message: Update mybot.xacro

File: nd_2w_4Dof/mybot_description/urdf/mybot.xacro (robot description, xacro)
@@ -244,5 +244,5 @@
         <child link="link_51" />
         <axis xyz="1 0 0" />
-        <limit lower="0" upper="0.4" effort="300" velocity="1" />
+        <limit lower="0" upper="0.4" effort="1" velocity="1" />
     </joint>
     <link name="link_52">
@@ -273,5 +273,5 @@
         <child link="link_52" />
         <axis xyz="1 0 0" />
-        <limit lower="-0.4" upper="0" effort="300" velocity="1" />
+        <limit lower="-0.4" upper="0" effort="1" velocity="1" />
     </joint>
     <transmission name="trans_joint_1">
