Commit message: Add files via upload

File: nd_2w_4Dof/tu_nguyen/urdf/tu_nguyen.urdf (robot description, URDF)
Before this commit: robot tu_nguyen, 7 links, 6 joints
Joints:
- joint joint_51: limit lower=0 upper=0.4 effort=300 velocity=1 -> lower=0 upper=0.4 effort=1 velocity=1
- joint joint_52: limit lower=-0.4 upper=0 effort=300 velocity=1 -> lower=-0.4 upper=0 effort=1 velocity=1
